Commit message: Move arm lower, make rail longer

File: osrf_gear/launch/linear_arm_actuator/linear_arm_actuator.urdf.xacro (robot description, xacro)
@@ -2,5 +2,5 @@
 <robot xmlns:xacro="http://www.ros.org/wiki/xacro">
 <xacro:property name="base_len" value="0.2" />
-<xacro:property name="actuator_len" value="4.6" />
+<xacro:property name="actuator_len" value="7.5" />
 <xacro:property name="actuator_height" value="0.1" />
 <xacro:arg name="use_velocity_interface" default="false" />

Commit message: Shorten belt to 4m again

File: osrf_gear/launch/linear_arm_actuator/linear_arm_actuator.urdf.xacro (robot description, xacro)
@@ -2,5 +2,5 @@
 <robot xmlns:xacro="http://www.ros.org/wiki/xacro">
 <xacro:property name="base_len" value="0.2" />
-<xacro:property name="actuator_len" value="7.5" />
+<xacro:property name="actuator_len" value="4.0" />
 <xacro:property name="actuator_height" value="0.1" />
 <xacro:arg name="use_velocity_interface" default="false" />
