Commit message: Fix xacro warnings

File: osrf_gear/vendor/ur_description/urdf/ur10.urdf.xacro (robot description, xacro)
@@ -10,5 +10,4 @@
   <!-- <xacro:include filename="$(find ur_description)/urdf/ur.gazebo.xacro" /> -->
   <xacro:include filename="$(find osrf_gear)/vendor/ur_description/urdf/ur.gazebo.xacro" />
-  <xacro:property name="pi" value="3.14159265" />
   <!-- Inertia parameters -->
   <xacro:property name="base_mass" value="4.0" />  <!-- This mass might be incorrect -->
