Commit message: Factor out product types

File: osrf_gear/launch/vacuum_gripper/vacuum_gripper.urdf.xacro (robot description, xacro)
@@ -1,5 +1,5 @@
 <?xml version="1.0"?>
 <robot xmlns:xacro="http://www.ros.org/wiki/xacro">
-<xacro:macro name="create_vacuum_gripper" params="wrist_link **drops_info">
+<xacro:macro name="create_vacuum_gripper" params="wrist_link **grippable_model_types **drops_info">
   <link name="vacuum_gripper_link">
     <inertial>
@@ -44,19 +44,5 @@
         <min_contact_count>1</min_contact_count>
       </grasp_check>
-      <grippable_model_types>
-        <type>part1</type>
-        <type>part2</type>
-        <type>part3</type>
-        <type>part4</type>
-        <type>arm_part</type>
-        <type>cross_joint_part</type>
-        <type>disk_part</type>
-        <type>gasket_part</type>
-        <type>gear_part</type>
-        <type>piston_rod_part</type>
-        <type>pulley_part</type>
-        <type>t_brace_part</type>
-        <type>u_joint_part</type>
-      </grippable_model_types>
+      <xacro:insert_block name="grippable_model_types" />
       <xacro:insert_block name="drops_info" />
       <suction_cup_link>vacuum_gripper_link</suction_cup_link>

Commit message: WIP gripper

File: osrf_gear/launch/vacuum_gripper/vacuum_gripper.urdf.xacro (robot description, xacro)
@@ -27,5 +27,5 @@
   </link>
   <joint name="vacuum_gripper_joint" type="revolute">
-    <origin xyz="0 0.1 0" rpy="${90 * 0.0174533} 0 0" />
+    <origin xyz="0 0.0 0.05" rpy="${0*90 * 0.0174533} 0 0" />
     <axis xyz="0 0 1" />
     <limit lower="0" upper="0" effort="0" velocity="0" />

Commit message: Origin as input to gripper

File: osrf_gear/launch/vacuum_gripper/vacuum_gripper.urdf.xacro (robot description, xacro)
@@ -1,5 +1,5 @@
 <?xml version="1.0"?>
 <robot xmlns:xacro="http://www.ros.org/wiki/xacro">
-<xacro:macro name="create_vacuum_gripper" params="wrist_link **grippable_model_types **drops_info">
+<xacro:macro name="create_vacuum_gripper" params="wrist_link *origin **grippable_model_types **drops_info">
   <link name="vacuum_gripper_link">
     <inertial>
@@ -27,5 +27,5 @@
   </link>
   <joint name="vacuum_gripper_joint" type="revolute">
-    <origin xyz="0 0.0 0.05" rpy="${0*90 * 0.0174533} 0 0" />
+    <xacro:insert_block name="origin" />
     <axis xyz="0 0 1" />
     <limit lower="0" upper="0" effort="0" velocity="0" />
