Commit message: Reduce max effort for other joints

File: osrf_gear/vendor/iiwa_description/urdf/iiwa14.xacro (robot description, xacro)
@@ -11,5 +11,5 @@
   <xacro:property name="safety_controller_k_vel" value="2" />
   <xacro:property name="joint_damping" value="0.5" />
-  <xacro:property name="max_effort" value="300"/>
+  <xacro:property name="max_effort" value="150"/>
   <xacro:property name="max_velocity" value="5"/>
   <xacro:macro name="iiwa14" params="parent hardware_interface robot_name *origin">

Commit message: Set joint damping to 0

File: osrf_gear/vendor/iiwa_description/urdf/iiwa14.xacro (robot description, xacro)
@@ -10,5 +10,5 @@
   <xacro:property name="safety_controller_k_pos" value="100" />
   <xacro:property name="safety_controller_k_vel" value="2" />
-  <xacro:property name="joint_damping" value="0.5" />
+  <xacro:property name="joint_damping" value="0.0" />
   <xacro:property name="max_effort" value="150"/>
   <xacro:property name="max_velocity" value="5"/>

Commit message: Revert "Merged in iiwa_effort_limits (pull request #96)"
This reverts commit f752b1ba423cce50bead3b554daeabd1bd9de8a2, reversing
changes made to a22cf9ca2446d57e76a68f53a150184af1e2e1fb.

File: osrf_gear/vendor/iiwa_description/urdf/iiwa14.xacro (robot description, xacro)
@@ -10,6 +10,6 @@
   <xacro:property name="safety_controller_k_pos" value="100" />
   <xacro:property name="safety_controller_k_vel" value="2" />
-  <xacro:property name="joint_damping" value="0.0" />
-  <xacro:property name="max_effort" value="150"/>
+  <xacro:property name="joint_damping" value="0.5" />
+  <xacro:property name="max_effort" value="300"/>
   <xacro:property name="max_velocity" value="5"/>
   <xacro:macro name="iiwa14" params="parent hardware_interface robot_name *origin">
@@ -266,5 +266,5 @@
       <axis xyz="0 0 1"/>
       <limit lower="${-175 * PI / 180}" upper="${175 * PI / 180}"
-             effort="5" velocity="${max_velocity}" />
+             effort="8" velocity="${max_velocity}" />
       <safety_controller soft_lower_limit="${-173 * PI / 180}"
                          soft_upper_limit="${173 * PI / 180}"
